File: compulator/compulator.kicad_pcb (KiCad board)
At the start: 2 copper layers, 58.4 x 63.5 mm, 47 parts, among them J1 S2B-PH-SM4-TB_LF__SN_, J2 S2B-PH-SM4-TB_LF__SN_, J3 S2B-PH-SM4-TB_LF__SN_, J4 Conn_01x06, P1 10k (2.4k), U1 Opamp_Dual, U4 TL074

Commit message: modified test pad names, flipped LED to bottom
Parts:
- D2: moved to B.Cu
- TP3: value OUT -> out
- TP4: value COMP_OUT -> comp
